File: garage_receiver.kicad_pcb (KiCad board)
At the start: 2 copper layers, 85 x 45 mm, 23 parts, among them J1 Conn_01x04_Female, J2 Screw_Terminal_01x04, Q1 2N7002, SW1 SW_DIP_x08, U1 HT12D, U2 LTC3255

Commit message: Label secret code switches and updated BOM
Other:
- board text added: "A0"
- board text added: "A1"
- board text added: "A2"
- board text added: "A3"
- board text added: "A4"
- board text added: "A5"
- board text added: "A6"
- board text added: "A7"
Changed lines of the file:
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@@
   (general
     (thickness 1.6)
-    (drawings 17)
+    (drawings 25)
     (tracks 129)
     (zones 0)
@@
     )
   )
+  (gr_text A6 (at 241.482 93.516) (layer F.SilkS)
+    (effects (font (size 1 1) (thickness 0.15)))
+  )
+  (gr_text A7 (at 241.482 90.916) (layer F.SilkS)
+    (effects (font (size 1 1) (thickness 0.15)))
+  )
+  (gr_text A4 (at 241.482 98.616) (layer F.SilkS)
+    (effects (font (size 1 1) (thickness 0.15)))
+  )
+  (gr_text A5 (at 241.482 96.016) (layer F.SilkS)
+    (effects (font (size 1 1) (thickness 0.15)))
+  )
+  (gr_text A2 (at 241.482 103.716) (layer F.SilkS)
+    (effects (font (size 1 1) (thickness 0.15)))
+  )
+  (gr_text A3 (at 241.482 101.116) (layer F.SilkS)
+    (effects (font (size 1 1) (thickness 0.15)))
+  )
+  (gr_text A1 (at 241.482 106.316) (layer F.SilkS)
+    (effects (font (size 1 1) (thickness 0.15)))
+  )
+  (gr_text A0 (at 241.482 108.916) (layer F.SilkS)
+    (effects (font (size 1 1) (thickness 0.15)))
+  )
   (gr_text "Garage Receiver" (at 191.782 115.216) (layer F.SilkS)

Commit message: Fixed Soldermask Clearance
Other:
- rule solder_mask_min_width: 0.25 -> 0.09
Changed lines of the file:
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@@
     (pad_drill 3.2)
     (pad_to_mask_clearance 0.051)
-    (solder_mask_min_width 0.25)
+    (solder_mask_min_width 0.09)
     (aux_axis_origin 0 0)
     (grid_origin 173.482 77.216)
