File: garage_receiver.kicad_pcb (KiCad board)
At the start: 2 copper layers, 85 x 45 mm, 23 parts, among them J1 Conn_01x04_Female, J2 Screw_Terminal_01x04, Q1 2N7002, SW1 SW_DIP_x08, U1 HT12D, U2 LTC3255

Commit message: Removed Undersized and Uneded  SMD Capacitor
Parts:
- removed C3: 1u, Capacitor_SMD:C_0805_2012Metric
Connections:
- H1 pad 1: GNDPWR -> (no net)
- H2 pad 1: GNDPWR -> (no net)
- H3 pad 1: GNDPWR -> (no net)
- H4 pad 1: GNDPWR -> (no net)
Routing:
- net GND: track 34.5 -> 30.4 mm
- net +36V: track 19.0 -> 15.1 mm
Other:
- board text added: "v1.0.1"
- board text removed: "v1.0.0"
