File: garage_receiver.sch (KiCad schematic (older format))
At the start: 23 parts, among them J1 Conn_01x04_Female, J2 Screw_Terminal_01x04, Q1 2N7002, SW1 SW_DIP_x08, U1 HT12D, U2 LTC3255

Commit message: Removed Undersized and Uneded  SMD Capacitor
Parts:
- removed C3: 1u, Capacitor_SMD:C_0805_2012Metric, symbol Device:C
Changed lines of the file:
@@
 	8650 4100 8650 4250
 Connection ~ 8650 4250
-$Comp
-L Device:C C3
-U 1 1 5D18053F
-P 6450 4500
-F 0 "C3" H 6565 4546 50  0000 L CNN
-F 1 "1u" H 6565 4455 50  0000 L CNN
-F 2 "Capacitor_SMD:C_0805_2012Metric" H 6488 4350 50  0001 C CNN
-F 3 "~" H 6450 4500 50  0001 C CNN
-	1    6450 4500
-	1    0    0    -1
-$EndComp
-Wire Wire Line
-	6450 4350 6450 3850
-Wire Wire Line
-	6450 3850 6700 3850
 Wire Wire Line
 	6700 4350 6700 3850
-Connection ~ 6700 3850
 Wire Wire Line
 	7650 3700 7650 3850
 Wire Wire Line
 	6700 4350 7150 4350
-Wire Wire Line
-	6450 4950 6850 4950
 Wire Wire Line
 	6700 3850 7650 3850
@@
 	1    0    0    -1
 $EndComp
-Wire Wire Line
-	6450 4650 6450 4950
 $Comp
 L Device:C C5
@@
 Wire Wire Line
 	6850 4450 6850 4950
-Connection ~ 6850 4950
 Wire Wire Line
 	6850 4950 7000 4950
